Commit message: Add a lidar frame

File: assets/h1_2/h1_2.urdf (robot description, URDF)
Before this commit: robot h1_2, 56 links, 55 joints
Links:
- added link lidar_link
Joints:
- added joint lidar_joint: type fixed, parent torso_link, child lidar_link, origin xyz=0.051307 0 0.68218 rpy=0 -2.88869 0

Commit message: Add a head camera frame

File: assets/h1_2/h1_2.urdf (robot description, URDF)
Before this commit: robot h1_2, 57 links, 56 joints
Links:
- added link head_camera_link
Joints:
- added joint head_camera_joint: type fixed, parent torso_link, child head_camera_link, origin xyz=0.11019 0.032508 0.68918 rpy=0 0.85811 0

Commit message: Sync urdf with added frames

File: assets/h1_2/h1_2.urdf (robot description, URDF)
Before this commit: robot h1_2, 58 links, 57 joints
Links:
- added link left_hand_camera_link
- added link right_hand_camera_link
Joints:
- added joint left_hand_camera_joint: type fixed, parent left_wrist_yaw_link, child left_hand_camera_link, origin xyz=0 0.04 0 rpy=0 1.5708 0
- added joint right_hand_camera_joint: type fixed, parent right_wrist_yaw_link, child right_hand_camera_link, origin xyz=0 -0.04 0 rpy=-3.1415 -1.5708 0
- joint head_camera_joint: origin xyz=0.11019 0.032508 0.68918 rpy=0 0.85811 0 -> xyz=0.11019 0.032508 0.68918 rpy=-2.42891 -0.00000278 -1.5708
